Commit message: add vellocity mode controllers.urdf.xacro

File: nekomimi_bot_description/urdf/controllers.urdf.xacro (robot description, xacro)
@@ -49,10 +49,10 @@
       </joint>
       <!-- Position Drive: Wheels -->
-      <!-- <joint name="left_wheel_joint">
+      <joint name="left_wheel_joint">
         <xacro:unless value="${$(arg enable_gz)}">
           <param name="initial_position">0.0</param>
           <param name="id">11</param>
-          <param name="p_cofficient">8</param>
-          <param name="offset">2048</param>
+          <!-- <param name="p_cofficient">8</param> -->
+          <!-- <param name="offset">2048</param> -->
         </xacro:unless>
         <command_interface name="velocity"/>
@@ -64,11 +64,11 @@
           <param name="initial_position">0.0</param>
           <param name="id">12</param>
-          <param name="p_cofficient">8</param>
-          <param name="offset">2048</param>
+          <!-- <param name="p_cofficient">8</param> -->
+          <!-- <param name="offset">2048</param> -->
         </xacro:unless>
         <command_interface name="velocity"/>
         <state_interface name="position"/>
         <state_interface name="velocity"/>
-      </joint> -->
+      </joint>
     </ros2_control>
     <!-- Ignition ROS2 Control -->
