Commit message: Add Navigation

File: nekomimi_bot_description/robots/nekomimi_bot_robot.urdf.xacro (robot description, xacro)
@@ -16,4 +16,5 @@
   <xacro:arg name="enable_gz"                 default="False" />
   <xacro:arg name="robot_name"                default="nekomimi_bot" />
+  <xacro:arg name="ftc_sl_port"               default="/dev/ttyUSB0" />
   <!-- Conection -->
   <xacro:base/>

File: nekomimi_bot_description/urdf/controllers.urdf.xacro (robot description, xacro)
@@ -8,6 +8,7 @@
         </xacro:if>
         <xacro:unless value="${$(arg enable_gz)}">
+          <xacro:property name="ftc_sl_port" value="$(arg ftc_sl_port)"/>
           <plugin>feetech_ros2_driver/FeetechHardwareInterface</plugin>
-          <param name="usb_port">/dev/ttyUSB0</param>
+          <param name="usb_port">${ftc_sl_port}</param>
         </xacro:unless>
       </hardware>
@@ -19,5 +20,5 @@
           <param name="p_cofficient">8</param>
           <param name="offset">2048</param>
-          <param name="counter_rotation">1</param>
+          <param name="counter_rotation">0</param>
         </xacro:unless>
         <command_interface name="position"/>
@@ -70,5 +71,5 @@
           <!-- <param name="p_cofficient">8</param> -->
           <!-- <param name="offset">2048</param> -->
-          <param name="counter_rotation">1</param>
+          <param name="counter_rotation">0</param>
         </xacro:unless>
         <command_interface name="velocity"/>

File: nekomimi_bot_description/urdf/mobile_base/wheel.urdf.xacro (robot description, xacro)
@@ -2,10 +2,10 @@
 <robot name="nekomimi_bot"
        xmlns:xacro="http://ros.org/wiki/xacro">
-  <xacro:macro name="wheel_base" params="parent prefix pose_y pose_yaw axis_y">
+  <xacro:macro name="wheel_base" params="parent prefix pose_yaw axis_y">
     <joint name="${prefix}_joint" type="continuous">
-      <origin xyz="0.0 ${pose_y} -0.01" rpy="0.0 0.0 0.0" />
+      <origin xyz="0.0 ${axis_y*0.0725} -0.01" rpy="0.0 0.0 0.0" />
       <parent link="${parent}" />
       <child link="${prefix}_link" />
-      <axis xyz="0.0 ${axis_y} 0.0 " />
+      <axis xyz="0.0 1.0 0.0 " />
       <limit effort="10.0" velocity="7.913672" />
     </joint>
@@ -34,6 +34,6 @@
   </xacro:macro>
   <xacro:macro name="wheel" params="parent prefix">
-    <xacro:wheel_base parent="${parent}_link" prefix="left_${prefix}"  pose_y="0.0725"  pose_yaw="${M_PI/2}"  axis_y="1.0"  />
-    <xacro:wheel_base parent="${parent}_link" prefix="right_${prefix}" pose_y="-0.0725" pose_yaw="${-M_PI/2}" axis_y="-1.0" />
+    <xacro:wheel_base parent="${parent}_link" prefix="left_${prefix}"  pose_yaw="${M_PI/2}"  axis_y="1.0"  />
+    <xacro:wheel_base parent="${parent}_link" prefix="right_${prefix}" pose_yaw="${-M_PI/2}" axis_y="-1.0" />
   </xacro:macro>
 </robot>

File: nekomimi_bot_description/urdf/mobile_base/wheel_base.urdf.xacro (robot description, xacro)
@@ -7,5 +7,5 @@
       <parent link="${parent}_link" />
       <child link="${prefix}_link" />
-      <axis xyz="0.0 0.0 -1.0 " />
+      <axis xyz="0.0 0.0 1.0 " />
       <limit lower="${-M_PI/2}" upper="${M_PI/2}" effort="4.1" velocity="4.796165" />
     </joint>
