Commit message: Comp

File: nekomimi_bot_description/urdf/body/body.urdf.xacro (robot description, xacro)
@@ -17,7 +17,8 @@
       </visual>
       <collision>
-        <origin xyz="0.0 0.0 0.0" rpy="0.0 0.0 0.0" />
+        <origin xyz="0.0 0.0 0.0" rpy="0.0 0.0 ${M_PI/2}" />
         <geometry>
-          <box size="0.1 0.1 0.1" />
+          <!-- <box size="0.1 0.1 0.1" /> -->
+          <mesh filename="file://$(find nekomimi_bot_description)/meshes/body/body_plate.stl" scale="0.001 0.001 0.001" />
         </geometry>
       </collision>
@@ -44,7 +45,8 @@
       </visual>
       <collision>
-        <origin xyz="0.0 0.0 0.0" rpy="0.0 0.0 0.0" />
+        <origin xyz="0.0 0.0 0.0" rpy="0.0 0.0 ${M_PI/2}" />
         <geometry>
-          <box size="0.1 0.1 0.1" />
+          <!-- <box size="0.1 0.1 0.1" /> -->
+          <mesh filename="file://$(find nekomimi_bot_description)/meshes/body/body_cover.stl" scale="0.001 0.001 0.001" />
         </geometry>
       </collision>

File: nekomimi_bot_description/urdf/controllers.urdf.xacro (robot description, xacro)
@@ -19,4 +19,5 @@
           <param name="p_cofficient">8</param>
           <param name="offset">2048</param>
+          <param name="counter_rotation">1</param>
         </xacro:unless>
         <command_interface name="position"/>
@@ -32,4 +33,5 @@
           <param name="p_cofficient">8</param>
           <param name="offset">2048</param>
+          <param name="counter_rotation">1</param>
         </xacro:unless>
         <command_interface name="position"/>
@@ -43,4 +45,5 @@
           <param name="p_cofficient">8</param>
           <param name="offset">2048</param>
+          <param name="counter_rotation">1</param>
         </xacro:unless>
         <command_interface name="position"/>
@@ -55,4 +58,5 @@
           <!-- <param name="p_cofficient">8</param> -->
           <!-- <param name="offset">2048</param> -->
+          <param name="counter_rotation">1</param>
         </xacro:unless>
         <command_interface name="velocity"/>
@@ -66,4 +70,5 @@
           <!-- <param name="p_cofficient">8</param> -->
           <!-- <param name="offset">2048</param> -->
+          <param name="counter_rotation">1</param>
         </xacro:unless>
         <command_interface name="velocity"/>

File: nekomimi_bot_description/urdf/head/head.urdf.xacro (robot description, xacro)
@@ -19,5 +19,6 @@
         <origin xyz="0.0 0.0 0.0" rpy="0.0 0.0 0.0" />
         <geometry>
-          <box size="0.1 0.1 0.1" />
+          <!-- <box size="0.1 0.1 0.1" /> -->
+          <mesh filename="file://$(find nekomimi_bot_description)/meshes/head/head_base.stl" scale="0.001 0.001 0.001" />
         </geometry>
       </collision>
@@ -50,5 +51,6 @@
         <origin xyz="0.0 0.0 0.0" rpy="0.0 0.0 0.0" />
         <geometry>
-          <box size="0.1 0.1 0.1" />
+          <!-- <box size="0.1 0.1 0.1" /> -->
+          <mesh filename="file://$(find nekomimi_bot_description)/meshes/head/head_tilt_base.stl" scale="0.001 0.001 0.001" />
         </geometry>
       </collision>
@@ -81,5 +83,6 @@
         <origin xyz="0.0 0.0 0.0" rpy="0.0 0.0 0.0" />
         <geometry>
-          <box size="0.1 0.1 0.1" />
+          <!-- <box size="0.1 0.1 0.1" /> -->
+          <mesh filename="file://$(find nekomimi_bot_description)/meshes/head/camera_base.stl" scale="0.001 0.001 0.001" />
         </geometry>
       </collision>

File: nekomimi_bot_description/urdf/mobile_base/wheel.urdf.xacro (robot description, xacro)
@@ -19,7 +19,7 @@
       </visual>
       <collision>
-        <origin xyz="0.0 0.0 0.0" rpy="0.0 0.0 0.0" />
+        <origin xyz="0.0 ${axis_y*0.0025} 0.0" rpy="${axis_y*M_PI/2} 0.0 0.0" />
         <geometry>
-          <box size="0.1 0.1 0.1" />
+          <cylinder radius="0.025" length="0.01"/>
         </geometry>
       </collision>

File: nekomimi_bot_description/urdf/mobile_base/wheel_base.urdf.xacro (robot description, xacro)
@@ -7,5 +7,5 @@
       <parent link="${parent}_link" />
       <child link="${prefix}_link" />
-      <axis xyz="0.0 0.0 1.0 " />
+      <axis xyz="0.0 0.0 -1.0 " />
       <limit lower="${-M_PI/2}" upper="${M_PI/2}" effort="4.1" velocity="4.796165" />
     </joint>
@@ -19,7 +19,8 @@
       </visual>
       <collision>
-        <origin xyz="0.0 0.0 0.0" rpy="0.0 0.0 0.0" />
+        <origin xyz="0.0 0.0 0.0" rpy="0.0 0.0 ${M_PI/2}" />
         <geometry>
-          <box size="0.1 0.1 0.1" />
+          <!-- <box size="0.1 0.1 0.1" /> -->
+          <mesh filename="file://$(find nekomimi_bot_description)/meshes/mobile_base/wheel_controller_core.stl" scale="0.001 0.001 0.001" />
         </geometry>
       </collision>

Commit message: Update mesh file of compress

File: nekomimi_bot_description/urdf/body/body.urdf.xacro (robot description, xacro)
@@ -12,16 +12,15 @@
         <origin xyz="0.0 0.0 0.0" rpy="0.0 0.0 ${M_PI/2}" />
         <geometry>
-          <mesh filename="file://$(find nekomimi_bot_description)/meshes/body/body_plate.stl" scale="0.001 0.001 0.001" />
+          <mesh filename="file://$(find nekomimi_bot_description)/meshes/body/body_core.stl" scale="0.001 0.001 0.001" />
         </geometry>
         <material name="black" />
       </visual>
       <collision>
-        <origin xyz="0.0 0.0 0.0" rpy="0.0 0.0 ${M_PI/2}" />
+        <origin xyz="0.0 0.0 0.0" rpy="0.0 0.0 0.0" />
         <geometry>
-          <!-- <box size="0.1 0.1 0.1" /> -->
-          <mesh filename="file://$(find nekomimi_bot_description)/meshes/body/body_plate.stl" scale="0.001 0.001 0.001" />
+          <cylinder radius="0.1" length="0.03"/>
         </geometry>
       </collision>
-      <inertial>
+      <!-- <inertial>
         <origin xyz="0.0 0.0 0.0" rpy="0.0 0.0 0.0" />
         <mass value="1.0" />
@@ -29,5 +28,5 @@
                  iyy="0.083" iyz="0.0"
                  izz="0.001" />
-      </inertial>
+      </inertial> -->
     </link>
     <joint name="${prefix}_cover_joint" type="fixed">
@@ -44,8 +43,7 @@
         <material name="black" />
       </visual>
-      <collision>
+      <!-- <collision>
         <origin xyz="0.0 0.0 0.0" rpy="0.0 0.0 ${M_PI/2}" />
         <geometry>
-          <!-- <box size="0.1 0.1 0.1" /> -->
           <mesh filename="file://$(find nekomimi_bot_description)/meshes/body/body_cover.stl" scale="0.001 0.001 0.001" />
         </geometry>
@@ -57,5 +55,5 @@
                  iyy="0.083" iyz="0.0"
                  izz="0.001" />
-      </inertial>
+      </inertial> -->
     </link>
   </xacro:macro>

File: nekomimi_bot_description/urdf/head/head.urdf.xacro (robot description, xacro)
@@ -16,9 +16,8 @@
         <material name="black" />
       </visual>
-      <collision>
+      <!-- <collision>
         <origin xyz="0.0 0.0 0.0" rpy="0.0 0.0 0.0" />
         <geometry>
-          <!-- <box size="0.1 0.1 0.1" /> -->
-          <mesh filename="file://$(find nekomimi_bot_description)/meshes/head/head_base.stl" scale="0.001 0.001 0.001" />
+          <box size="0.1 0.1 0.1" />
         </geometry>
       </collision>
@@ -29,5 +28,5 @@
                  iyy="0.083" iyz="0.0"
                  izz="0.001" />
-      </inertial>
+      </inertial> -->
     </link>
   </xacro:macro>
@@ -48,9 +47,8 @@
         <material name="black" />
       </visual>
-      <collision>
+      <!-- <collision>
         <origin xyz="0.0 0.0 0.0" rpy="0.0 0.0 0.0" />
         <geometry>
-          <!-- <box size="0.1 0.1 0.1" /> -->
-          <mesh filename="file://$(find nekomimi_bot_description)/meshes/head/head_tilt_base.stl" scale="0.001 0.001 0.001" />
+          <box size="0.1 0.1 0.1" />
         </geometry>
       </collision>
@@ -61,5 +59,5 @@
                  iyy="0.083" iyz="0.0"
                  izz="0.001" />
-      </inertial>
+      </inertial> -->
     </link>
   </xacro:macro>
@@ -80,9 +78,8 @@
         <material name="black" />
       </visual>
-      <collision>
+      <!-- <collision>
         <origin xyz="0.0 0.0 0.0" rpy="0.0 0.0 0.0" />
         <geometry>
-          <!-- <box size="0.1 0.1 0.1" /> -->
-          <mesh filename="file://$(find nekomimi_bot_description)/meshes/head/camera_base.stl" scale="0.001 0.001 0.001" />
+          <box size="0.1 0.1 0.1" />
         </geometry>
       </collision>
@@ -93,5 +90,5 @@
                  iyy="0.083" iyz="0.0"
                  izz="0.001" />
-      </inertial>
+      </inertial> -->
     </link>
   </xacro:macro>

File: nekomimi_bot_description/urdf/mobile_base/wheel.urdf.xacro (robot description, xacro)
@@ -24,5 +24,5 @@
         </geometry>
       </collision>
-      <inertial>
+      <!-- <inertial>
         <origin xyz="0.0 0.0 0.0" rpy="0.0 0.0 0.0" />
         <mass value="1.0" />
@@ -30,5 +30,5 @@
                  iyy="0.083" iyz="0.0"
                  izz="0.001" />
-      </inertial>
+      </inertial> -->
     </link>
   </xacro:macro>

File: nekomimi_bot_description/urdf/mobile_base/wheel_base.urdf.xacro (robot description, xacro)
@@ -18,9 +18,8 @@
         <material name="black" />
       </visual>
-      <collision>
+      <!-- <collision>
         <origin xyz="0.0 0.0 0.0" rpy="0.0 0.0 ${M_PI/2}" />
         <geometry>
-          <!-- <box size="0.1 0.1 0.1" /> -->
-          <mesh filename="file://$(find nekomimi_bot_description)/meshes/mobile_base/wheel_controller_core.stl" scale="0.001 0.001 0.001" />
+          <box size="0.1 0.1 0.1" />
         </geometry>
       </collision>
@@ -31,5 +30,5 @@
                  iyy="0.083" iyz="0.0"
                  izz="0.001" />
-      </inertial>
+      </inertial> -->
     </link>
   </xacro:macro>

File: nekomimi_bot_description/urdf/sensor/camera.urdf.xacro (robot description, xacro)
@@ -5,5 +5,4 @@
     <joint name="realsense_d405" type="fixed">
       <origin xyz="-0.00982012 0.0 0.0305" rpy="0.0 0.0 0.0" />
-      <!-- <origin xyz="-0.00982012 0.0 0.0515" rpy="0.0 0.0 0.0" /> -->
       <parent link="${parent}_link" />
       <child link="realsense_link" />
@@ -12,5 +11,4 @@
       <visual>
         <origin xyz="0.02293 0.0 0.021" rpy="${M_PI/2} 0.0 ${M_PI/2}" />
-        <!-- <origin xyz="0.02293 0.0 0.0" rpy="${M_PI/2} 0.0 ${M_PI/2}" /> -->
         <geometry>
           <mesh filename="file://$(find nekomimi_bot_description)/meshes/sensor/realsense_d405.stl" scale="0.001 0.001 0.001" />
@@ -18,5 +16,5 @@
         <material name="grey" />
       </visual>
-      <collision>
+      <!-- <collision>
         <origin xyz="0.0 0.0 0.0" rpy="0.0 0.0 0.0" />
         <geometry>
@@ -30,5 +28,5 @@
                  iyy="0.083" iyz="0.0"
                  izz="0.001" />
-      </inertial>
+      </inertial> -->
     </link>
   </xacro:macro>

File: nekomimi_bot_description/urdf/sensor/lidar.urdf.xacro (robot description, xacro)
@@ -16,5 +16,5 @@
         <material name="dark_grey" />
       </visual>
-      <collision>
+      <!-- <collision>
         <origin xyz="0.0 0.0 0.0" rpy="0.0 0.0 0.0" />
         <geometry>
@@ -28,5 +28,5 @@
                  iyy="0.083" iyz="0.0"
                  izz="0.001" />
-      </inertial>
+      </inertial> -->
     </link>
   </xacro:macro>

Commit message: update 3d model from cad(compress data)

File: nekomimi_bot_description/urdf/body/body.urdf.xacro (robot description, xacro)
@@ -17,16 +17,22 @@
       </visual>
       <collision>
-        <origin xyz="0.0 0.0 0.0" rpy="0.0 0.0 0.0" />
+        <origin xyz="0.0 0.0 0.017" rpy="0.0 0.0 0.0" />
         <geometry>
-          <cylinder radius="0.1" length="0.03"/>
+          <cylinder radius="0.0982680435950569" length="0.070"/>
         </geometry>
       </collision>
-      <!-- <inertial>
+      <collision>
+        <origin xyz="0.0 0.0 0.105" rpy="0.0 0.0 0.0" />
+        <geometry>
+          <box size="0.02 0.145 0.112" />
+        </geometry>
+      </collision>
+      <inertial>
         <origin xyz="0.0 0.0 0.0" rpy="0.0 0.0 0.0" />
         <mass value="1.0" />
-        <inertia ixx="0.083" ixy="0.0" ixz="0.0"
-                 iyy="0.083" iyz="0.0"
-                 izz="0.001" />
-      </inertial> -->
+        <inertia ixx="0.001" ixy="0.0" ixz="0.0"
+                 iyy="0.001" iyz="0.0"
+                 izz="0.001"/>
+      </inertial>
     </link>
     <joint name="${prefix}_cover_joint" type="fixed">
@@ -43,17 +49,4 @@
         <material name="black" />
       </visual>
-      <!-- <collision>
-        <origin xyz="0.0 0.0 0.0" rpy="0.0 0.0 ${M_PI/2}" />
-        <geometry>
-          <mesh filename="file://$(find nekomimi_bot_description)/meshes/body/body_cover.stl" scale="0.001 0.001 0.001" />
-        </geometry>
-      </collision>
-      <inertial>
-        <origin xyz="0.0 0.0 0.0" rpy="0.0 0.0 0.0" />
-        <mass value="1.0" />
-        <inertia ixx="0.083" ixy="0.0" ixz="0.0"
-                 iyy="0.083" iyz="0.0"
-                 izz="0.001" />
-      </inertial> -->
     </link>
   </xacro:macro>

File: nekomimi_bot_description/urdf/head/head.urdf.xacro (robot description, xacro)
@@ -16,8 +16,8 @@
         <material name="black" />
       </visual>
-      <!-- <collision>
-        <origin xyz="0.0 0.0 0.0" rpy="0.0 0.0 0.0" />
+      <collision>
+        <origin xyz="-0.00529 0.0 0.035" rpy="0.0 0.0 0.0" />
         <geometry>
-          <box size="0.1 0.1 0.1" />
+          <box size="0.032 0.021 0.069" />
         </geometry>
       </collision>
@@ -25,8 +25,8 @@
         <origin xyz="0.0 0.0 0.0" rpy="0.0 0.0 0.0" />
         <mass value="1.0" />
-        <inertia ixx="0.083" ixy="0.0" ixz="0.0"
-                 iyy="0.083" iyz="0.0"
-                 izz="0.001" />
-      </inertial> -->
+        <inertia ixx="0.001" ixy="0.0" ixz="0.0"
+                 iyy="0.001" iyz="0.0"
+                 izz="0.001"/>
+      </inertial>
     </link>
   </xacro:macro>
@@ -47,17 +47,11 @@
         <material name="black" />
       </visual>
-      <!-- <collision>
-        <origin xyz="0.0 0.0 0.0" rpy="0.0 0.0 0.0" />
-        <geometry>
-          <box size="0.1 0.1 0.1" />
-        </geometry>
-      </collision>
       <inertial>
         <origin xyz="0.0 0.0 0.0" rpy="0.0 0.0 0.0" />
         <mass value="1.0" />
-        <inertia ixx="0.083" ixy="0.0" ixz="0.0"
-                 iyy="0.083" iyz="0.0"
-                 izz="0.001" />
-      </inertial> -->
+        <inertia ixx="0.001" ixy="0.0" ixz="0.0"
+                 iyy="0.001" iyz="0.0"
+                 izz="0.001"/>
+      </inertial>
     </link>
   </xacro:macro>
@@ -78,17 +72,4 @@
         <material name="black" />
       </visual>
-      <!-- <collision>
-        <origin xyz="0.0 0.0 0.0" rpy="0.0 0.0 0.0" />
-        <geometry>
-          <box size="0.1 0.1 0.1" />
-        </geometry>
-      </collision>
-      <inertial>
-        <origin xyz="0.0 0.0 0.0" rpy="0.0 0.0 0.0" />
-        <mass value="1.0" />
-        <inertia ixx="0.083" ixy="0.0" ixz="0.0"
-                 iyy="0.083" iyz="0.0"
-                 izz="0.001" />
-      </inertial> -->
     </link>
   </xacro:macro>

File: nekomimi_bot_description/urdf/mobile_base/wheel.urdf.xacro (robot description, xacro)
@@ -24,11 +24,11 @@
         </geometry>
       </collision>
-      <!-- <inertial>
+      <inertial>
         <origin xyz="0.0 0.0 0.0" rpy="0.0 0.0 0.0" />
         <mass value="1.0" />
-        <inertia ixx="0.083" ixy="0.0" ixz="0.0"
-                 iyy="0.083" iyz="0.0"
-                 izz="0.001" />
-      </inertial> -->
+        <inertia ixx="0.001" ixy="0.0" ixz="0.0"
+                 iyy="0.001" iyz="0.0"
+                 izz="0.001"/>
+      </inertial>
     </link>
   </xacro:macro>

File: nekomimi_bot_description/urdf/mobile_base/wheel_base.urdf.xacro (robot description, xacro)
@@ -18,8 +18,14 @@
         <material name="black" />
       </visual>
-      <!-- <collision>
-        <origin xyz="0.0 0.0 0.0" rpy="0.0 0.0 ${M_PI/2}" />
+      <collision>
+        <origin xyz="0.062 0.0 -0.02" rpy="0.0 0.0 0.0" />
         <geometry>
-          <box size="0.1 0.1 0.1" />
+          <sphere radius="0.0146"/>
+        </geometry>
+      </collision>
+      <collision>
+        <origin xyz="-0.062 0.0 -0.02" rpy="0.0 0.0 0.0" />
+        <geometry>
+          <sphere radius="0.0146"/>
         </geometry>
       </collision>
@@ -27,8 +33,8 @@
         <origin xyz="0.0 0.0 0.0" rpy="0.0 0.0 0.0" />
         <mass value="1.0" />
-        <inertia ixx="0.083" ixy="0.0" ixz="0.0"
-                 iyy="0.083" iyz="0.0"
-                 izz="0.001" />
-      </inertial> -->
+        <inertia ixx="0.001" ixy="0.0" ixz="0.0"
+                 iyy="0.001" iyz="0.0"
+                 izz="0.001"/>
+      </inertial>
     </link>
   </xacro:macro>

File: nekomimi_bot_description/urdf/sensor/camera.urdf.xacro (robot description, xacro)
@@ -16,8 +16,8 @@
         <material name="grey" />
       </visual>
-      <!-- <collision>
-        <origin xyz="0.0 0.0 0.0" rpy="0.0 0.0 0.0" />
+      <collision>
+        <origin xyz="0.0135 0.0 0.0245" rpy="0.0 0.0 0.0" />
         <geometry>
-          <box size="0.1 0.1 0.1" />
+          <box size="0.027 0.049 0.049" />
         </geometry>
       </collision>
@@ -25,8 +25,8 @@
         <origin xyz="0.0 0.0 0.0" rpy="0.0 0.0 0.0" />
         <mass value="1.0" />
-        <inertia ixx="0.083" ixy="0.0" ixz="0.0"
-                 iyy="0.083" iyz="0.0"
-                 izz="0.001" />
-      </inertial> -->
+        <inertia ixx="0.001" ixy="0.0" ixz="0.0"
+                 iyy="0.001" iyz="0.0"
+                 izz="0.001"/>
+      </inertial>
     </link>
   </xacro:macro>

File: nekomimi_bot_description/urdf/sensor/lidar.urdf.xacro (robot description, xacro)
@@ -16,8 +16,8 @@
         <material name="dark_grey" />
       </visual>
-      <!-- <collision>
-        <origin xyz="0.0 0.0 0.0" rpy="0.0 0.0 0.0" />
+      <collision>
+        <origin xyz="0.0 0.0 -0.0072" rpy="0.0 0.0 0.0" />
         <geometry>
-          <box size="0.1 0.1 0.1" />
+          <cylinder radius="0.0325" length="0.0271"/>
         </geometry>
       </collision>
@@ -25,8 +25,8 @@
         <origin xyz="0.0 0.0 0.0" rpy="0.0 0.0 0.0" />
         <mass value="1.0" />
-        <inertia ixx="0.083" ixy="0.0" ixz="0.0"
-                 iyy="0.083" iyz="0.0"
-                 izz="0.001" />
-      </inertial> -->
+        <inertia ixx="0.001" ixy="0.0" ixz="0.0"
+                 iyy="0.001" iyz="0.0"
+                 izz="0.001"/>
+      </inertial>
     </link>
   </xacro:macro>
