Commit message: [TRY] Robot State Publisher path is not expansion to Multi PC

File: nekomimi_bot_description/urdf/body/body.urdf.xacro (robot description, xacro)
@@ -12,5 +12,5 @@
         <origin xyz="0.0 0.0 0.0" rpy="0.0 0.0 ${M_PI/2}" />
         <geometry>
-          <mesh filename="file://$(find nekomimi_bot_description)/meshes/body/body_core.stl" scale="0.001 0.001 0.001" />
+          <mesh filename="package://nekomimi_bot_description/meshes/body/body_core.stl" scale="0.001 0.001 0.001" />
         </geometry>
         <material name="black" />
@@ -45,5 +45,5 @@
         <origin xyz="0.0 0.0 0.0" rpy="0.0 0.0 ${M_PI/2}" />
         <geometry>
-          <mesh filename="file://$(find nekomimi_bot_description)/meshes/body/body_cover.stl" scale="0.001 0.001 0.001" />
+          <mesh filename="package://nekomimi_bot_description/meshes/body/body_cover.stl" scale="0.001 0.001 0.001" />
         </geometry>
         <material name="black" />

File: nekomimi_bot_description/urdf/head/head.urdf.xacro (robot description, xacro)
@@ -12,5 +12,5 @@
         <origin xyz="0.0 0.0 0.0" rpy="0.0 0.0 ${M_PI/2}" />
         <geometry>
-          <mesh filename="file://$(find nekomimi_bot_description)/meshes/head/head_base.stl" scale="0.001 0.001 0.001" />
+          <mesh filename="package://nekomimi_bot_description/meshes/head/head_base.stl" scale="0.001 0.001 0.001" />
         </geometry>
         <material name="black" />
@@ -43,5 +43,5 @@
         <origin xyz="0.0 0.0 0.0" rpy="0.0 0.0 ${M_PI/2}" />
         <geometry>
-          <mesh filename="file://$(find nekomimi_bot_description)/meshes/head/head_tilt_base.stl" scale="0.001 0.001 0.001" />
+          <mesh filename="package://nekomimi_bot_description/meshes/head/head_tilt_base.stl" scale="0.001 0.001 0.001" />
         </geometry>
         <material name="black" />
@@ -68,5 +68,5 @@
         <origin xyz="0.0 0.0 0.0" rpy="0.0 0.0 ${M_PI/2}" />
         <geometry>
-          <mesh filename="file://$(find nekomimi_bot_description)/meshes/head/camera_base.stl" scale="0.001 0.001 0.001" />
+          <mesh filename="package://nekomimi_bot_description/meshes/head/camera_base.stl" scale="0.001 0.001 0.001" />
         </geometry>
         <material name="black" />

File: nekomimi_bot_description/urdf/mobile_base/wheel.urdf.xacro (robot description, xacro)
@@ -14,5 +14,5 @@
         <origin xyz="0.0 0.0 0.0" rpy="0.0 0.0 ${pose_yaw}" />
         <geometry>
-          <mesh filename="file://$(find nekomimi_bot_description)/meshes/mobile_base/wheel.stl" scale="0.001 0.001 0.001" />
+          <mesh filename="package://nekomimi_bot_description/meshes/mobile_base/wheel.stl" scale="0.001 0.001 0.001" />
         </geometry>
         <material name="wheel" />

File: nekomimi_bot_description/urdf/mobile_base/wheel_base.urdf.xacro (robot description, xacro)
@@ -14,5 +14,5 @@
         <origin xyz="0.0 0.0 0.0" rpy="0.0 0.0 ${M_PI/2}" />
         <geometry>
-          <mesh filename="file://$(find nekomimi_bot_description)/meshes/mobile_base/wheel_controller_core.stl" scale="0.001 0.001 0.001" />
+          <mesh filename="package://nekomimi_bot_description/meshes/mobile_base/wheel_controller_core.stl" scale="0.001 0.001 0.001" />
         </geometry>
         <material name="black" />

File: nekomimi_bot_description/urdf/sensor/camera.urdf.xacro (robot description, xacro)
@@ -12,5 +12,5 @@
         <origin xyz="-0.00007 -0.009 ${0.021-0.021}" rpy="${M_PI/2} 0.0 ${M_PI/2}" />
         <geometry>
-          <mesh filename="file://$(find nekomimi_bot_description)/meshes/sensor/realsense_d405.stl" scale="0.001 0.001 0.001" />
+          <mesh filename="package://nekomimi_bot_description/meshes/sensor/realsense_d405.stl" scale="0.001 0.001 0.001" />
         </geometry>
         <material name="grey" />

File: nekomimi_bot_description/urdf/sensor/lidar.urdf.xacro (robot description, xacro)
@@ -12,5 +12,5 @@
         <origin xyz="0.0 0.0 -0.02215" rpy="0.0 0.0 0.0" />
         <geometry>
-          <mesh filename="file://$(find nekomimi_bot_description)/meshes/sensor/lds_lidar.stl" scale="0.001 0.001 0.001" />
+          <mesh filename="package://nekomimi_bot_description/meshes/sensor/lds_lidar.stl" scale="0.001 0.001 0.001" />
         </geometry>
         <material name="dark_grey" />
