Commit message: [UPD&ADD] src and realsense for lyrical

File: nekomimi_bot_description/urdf/head/head.urdf.xacro (robot description, xacro)
@@ -37,5 +37,5 @@
       <child link="${prefix}_link" />
       <axis xyz="0.0 0.0 1.0 " />
-      <limit lower="${-M_PI/2}" upper="${M_PI/2}" effort="4.1" velocity="4.796165" />
+      <limit lower="${-M_PI/2}" upper="${M_PI}" effort="4.1" velocity="4.796165" />
     </joint>
     <link name="${prefix}_link">
@@ -62,5 +62,5 @@
       <child link="${prefix}_link" />
       <axis xyz="0.0 1.0 0.0 " />
-      <limit lower="${-M_PI/2}" upper="${M_PI/2}" effort="4.1" velocity="4.796165" />
+      <limit lower="${-2*M_PI/3}" upper="${2*M_PI/3}" effort="4.1" velocity="4.796165" />
     </joint>
     <link name="${prefix}_link">
